File: BigClown_WiFi_module.brd (EAGLE design)
At the start: 100 x 80 mm, 17 parts

Commit message: Add files via upload
new version of design
Parts:
- moved R2 10.3 mm to (25.7, 37.7), flipped to the bottom
- moved R1 10.2 mm to (21.0, 41.9), flipped to the bottom
- moved R6 10.2 mm to (23.2, 41.9), flipped to the bottom
- moved R5 10.2 mm to (25.7, 41.9), flipped to the bottom
- moved C2 7.75 mm to (24.3, 32.5), turned to 0 degrees
- moved C1 7.24 mm to (24.4, 29.1), turned to 0 degrees
- moved IO2 1.31 mm to (33.0, 25.9)
- moved R3 0.64 mm to (32.3, 31.1)
- moved R4 0.63 mm to (32.3, 29.0)
- moved RST 0.54 mm to (32.8, 33.4)
Routing:
- net GND: track 79.6 -> 66.1 mm, vias 2 -> 4
- net N$1: track 19.6 -> 10.2 mm, vias 0 -> 1
- net VCC: track 64.9 -> 71.8 mm, vias 0 -> 1
- net CH_PD: track 17.4 -> 23.7 mm, vias 2 -> 1
- net N$2: track 19.5 -> 20.8 mm
- net RESET: track 55.3 -> 54.3 mm, vias 4 -> 1
- net N$3: track 9.59 -> 10.3 mm
- net N$4: track 37.0 -> 36.4 mm

Commit message: Add files via upload
Parts:
- moved RESET 5.80 mm to (14.9, 30.7)
- moved CH_PD 5.71 mm to (14.9, 26.7)
- moved C2 5.33 mm to (24.3, 27.2)
- moved R4 2.16 mm to (32.3, 26.8)
- moved IO2 1.91 mm to (33.1, 24.0)
- moved RST 1.66 mm to (32.9, 31.8)
- moved R3 1.65 mm to (32.3, 29.5)
- moved C1 1.40 mm to (24.3, 30.5)
Routing:
- net RESET: track 54.3 -> 48.6 mm
- net CH_PD: track 23.7 -> 18.7 mm
- net VCC: track 71.8 -> 67.4 mm
- net GND: track 66.1 -> 68.0 mm
- net N$3: track 10.3 -> 11.9 mm
- net N$2: track 20.8 -> 22.4 mm
- net P6: track 2.48 -> 4.04 mm
- net N$4: track 36.4 -> 37.7 mm
- net P7: track 2.48 -> 3.66 mm
- net P9: track 2.48 -> 3.62 mm
- net P8: track 2.48 -> 3.62 mm

Commit message: Add files via upload
Routing:
- net GND: track 68.0 -> 60.2 mm, vias 4 -> 2

Commit message: Add files via upload
Routing:
- net GND: track 60.2 -> 59.6 mm, vias 2 -> 1

Commit message: Add files via upload
Parts:
- removed IO2, RST: PTR1PAD1-13, testpad:P1-13
- added U$2, U$3, U$4, U$5, U$6, U$7, U$8: 1X1, headers_2mm:1X1
Connections:
- new net N$10: U$1.GPIO2, U$8.1
- new net N$6: U$1.GPIO12, U$5.1
- new net N$7: U$1.GPIO14, U$4.1
- new net N$8: U$1.GPIO4, U$6.1
- new net N$9: U$1.GPIO5, U$7.1
- net N$2: now also U$2.1; no longer IO2.TP
- net N$4: now also U$3.1; no longer RST.TP
- net RX: now also JP3.3; no longer JP3.1
- net TX: now also JP3.4; no longer JP3.2
Routing:
- net N$4: track 37.7 -> 23.5 mm
- net N$10: track 0.00 -> 11.8 mm, vias 0 -> 1
- net N$6: track 0.00 -> 3.16 mm
- net N$7: track 0.00 -> 2.69 mm
- net N$9: track 0.00 -> 2.49 mm
- net N$8: track 0.00 -> 2.48 mm
- net TX: track 24.6 -> 27.0 mm
- net RX: track 21.0 -> 23.0 mm
Other:
- board text added: "IO0"
- board text added: "IO12"
- board text added: "IO14"
- board text added: "IO2"
- board text added: "IO4"
- board text added: "IO5"
- board text added: "RST"

Commit message: v1.0
added pins for gpio
added labels
Parts:
- moved U$1 0.25 mm to (24.4, 44.5)
Other:
- board text added: "BigClown."
- board text added: "Made by"
- board text added: "WiFi module for"
- board text added: "v1.0 (6/2018)"

Commit message: Add files via upload
Parts:
- removed JP3: BC-MODULE-CORE, bigclown:BC-MODULE-CORE
- added JP2: BC-HEADER-MODULE-THT, bc-header:BC-HEADER-MODULE-THT
- R1: value 10k -> 1k
- renumbered U$2 to IO0, U$3 to RST, U$4 to IO14, U$5 to IO12, U$6 to IO4, U$7 to IO5, U$8 to IO2
Connections:
- net GND: now also JP2.15; no longer JP3.15
- net P6: now also JP2.7; no longer JP3.7
- net P7: now also JP2.8; no longer JP3.8
- net P8: now also JP2.9; no longer JP3.9
- net P9: now also JP2.10; no longer JP3.10
- net RX: now also JP2.3; no longer JP3.3
- net TX: now also JP2.4; no longer JP3.4
- net VCC: now also JP2.16; no longer JP3.16
Routing:
- net N$4: track 23.5 -> 22.9 mm
