File: BigClown_WiFi_module.sch (EAGLE design)
At the start: 17 parts

Commit message: Add files via upload
Parts:
- removed IO2, RST: PTR1PAD1-13, testpad:PTR1PAD1-13
- added U$2, U$3, U$4, U$5, U$6, U$7, U$8: 1X1, headers_2mm:1X1
Connections:
- new net N$10: U$1.GPIO2, U$8.1
- new net N$6: U$1.GPIO12, U$5.1
- new net N$7: U$1.GPIO14, U$4.1
- new net N$8: U$1.GPIO4, U$6.1
- new net N$9: U$1.GPIO5, U$7.1
- net N$2: now also U$2.1; no longer IO2.TP
- net N$4: now also U$3.1; no longer RST.TP
- net RX: now also JP3.P2/A2/TXD1; no longer JP3.P0/A0/TXD0
- net TX: now also JP3.P3/A3/RXD1; no longer JP3.P1/A1/RXD0
Changed lines of the file:
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@@
 <setting verticaltext="up"/>
 </settings>
-<grid distance="0.1" unitdist="inch" unit="inch" style="lines" multiple="1" display="no" altdistance="0.01" altunitdist="inch" altunit="inch"/>
+<grid distance="0.1" unitdist="inch" unit="mm" style="lines" multiple="1" display="no" altdistance="0.01" altunitdist="inch" altunit="inch"/>
 <layers>
 <layer number="1" name="Top" color="4" fill="1" visible="no" active="no"/>
@@
 <part name="RESET" library="SparkFun-Jumpers" library_urn="urn:adsk.eagle:library:528" deviceset="JUMPER-SMT_3_1-NC_PASTE" device="_SILK" package3d_urn="urn:adsk.eagle:package:39293/1"/>
 <part name="R5" library="rcl" library_urn="urn:adsk.eagle:library:334" deviceset="R-EU_" device="M0805" package3d_urn="urn:adsk.eagle:package:23556/1" value="10k"/>
-<part name="RST" library="testpad" library_urn="urn:adsk.eagle:library:385" deviceset="PTR1" device="PAD1-13" package3d_urn="urn:adsk.eagle:package:27946/1"/>
-<part name="IO2" library="testpad" library_urn="urn:adsk.eagle:library:385" deviceset="PTR1" device="PAD1-13" package3d_urn="urn:adsk.eagle:package:27946/1"/>
 <part name="R6" library="rcl" library_urn="urn:adsk.eagle:library:334" deviceset="R-EU_" device="M0805" package3d_urn="urn:adsk.eagle:package:23556/1" value="10k"/>
 <part name="P+6" library="supply1" library_urn="urn:adsk.eagle:library:371" deviceset="VCC" device=""/>
 <part name="JP1" library="SparkFun-Jumpers" library_urn="urn:adsk.eagle:library:528" deviceset="JUMPER-SMT_2_NO" device="_NO-SILK" package3d_urn="urn:adsk.eagle:package:39277/1"/>
+<part name="U$2" library="headers_2mm" deviceset="1X1" device=""/>
+<part name="U$3" library="headers_2mm" deviceset="1X1" device=""/>
+<part name="U$4" library="headers_2mm" deviceset="1X1" device=""/>
+<part name="U$5" library="headers_2mm" deviceset="1X1" device=""/>
+<part name="U$6" library="headers_2mm" deviceset="1X1" device=""/>
+<part name="U$7" library="headers_2mm" deviceset="1X1" device=""/>
+<part name="U$8" library="headers_2mm" deviceset="1X1" device=""/>
 </parts>
 <sheets>
@@
 <instance part="GND2" gate="1" x="121.92" y="40.64"/>
 <instance part="JP3" gate="JP" x="60.96" y="22.86"/>
-<instance part="P+1" gate="VCC" x="91.44" y="0"/>
+<instance part="P+1" gate="VCC" x="91.44" y="-2.54"/>
 <instance part="GND1" gate="1" x="91.44" y="-15.24"/>
 <instance part="CH_PD" gate="G$1" x="167.64" y="50.8" smashed="yes">
@@
 <instance part="U$1" gate="G$1" x="149.86" y="5.08"/>
 <instance part="GND3" gate="1" x="180.34" y="-10.16"/>
-<instance part="P+3" gate="VCC" x="106.68" y="0"/>
+<instance part="P+3" gate="VCC" x="106.68" y="-2.54"/>
 <instance part="S1" gate="G$1" x="208.28" y="5.08"/>
 <instance part="GND4" gate="1" x="203.2" y="-10.16"/>
@@
 </instance>
 <instance part="P+4" gate="VCC" x="203.2" y="27.94"/>
-<instance part="P+5" gate="VCC" x="182.88" y="10.16"/>
+<instance part="P+5" gate="VCC" x="195.58" y="5.08" smashed="yes">
+<attribute name="VALUE" x="198.12" y="-2.54" size="1.778" layer="96" rot="R90"/>
+</instance>
 <instance part="R3" gate="G$1" x="172.72" y="-2.54" smashed="yes" rot="R180">
 <attribute name="NAME" x="169.545" y="-0.2286" size="1.778" layer="95" rot="R180"/>
@@
 <attribute name="VALUE" x="117.475" y="10.668" size="1.778" layer="96"/>
 </instance>
-<instance part="RST" gate="G$1" x="132.08" y="17.78" rot="R180"/>
-<instance part="IO2" gate="G$1" x="167.64" y="17.78" rot="R180"/>
 <instance part="R6" gate="G$1" x="129.54" y="20.32" smashed="yes" rot="R90">
 <attribute name="NAME" x="129.3114" y="13.97" size="1.778" layer="95" rot="R90"/>
@@
 <attribute name="NAME" x="121.92" y="2.54" size="1.778" layer="95" font="vector"/>
 </instance>
+<instance part="U$2" gate="G$1" x="167.64" y="27.94" rot="R270"/>
+<instance part="U$3" gate="G$1" x="132.08" y="27.94" rot="R270"/>
+<instance part="U$4" gate="G$1" x="101.6" y="5.08" rot="R270"/>
+<instance part="U$5" gate="G$1" x="93.98" y="2.54" rot="R270"/>
+<instance part="U$6" gate="G$1" x="177.8" y="20.32" rot="R270"/>
+<instance part="U$7" gate="G$1" x="185.42" y="25.4" rot="R270"/>
+<instance part="U$8" gate="G$1" x="190.5" y="20.32" rot="R270"/>
 </instances>
 <busses>
@@
 <pinref part="P+1" gate="VCC" pin="VCC"/>
 <wire x1="83.82" y1="-5.08" x2="91.44" y2="-5.08" width="0.1524" layer="91"/>
-<wire x1="91.44" y1="-5.08" x2="91.44" y2="-2.54" width="0.1524" layer="91"/>
 </segment>
 <segment>
 <pinref part="U$1" gate="G$1" pin="VCC"/>
 <wire x1="132.08" y1="-5.08" x2="106.68" y2="-5.08" width="0.1524" layer="91"/>
-<wire x1="106.68" y1="-5.08" x2="106.68" y2="-2.54" width="0.1524" layer="91"/>
 <pinref part="P+3" gate="VCC" pin="VCC"/>
 </segment>
@@
 <segment>
 <pinref part="P+5" gate="VCC" pin="VCC"/>
-<wire x1="182.88" y1="2.54" x2="182.88" y2="7.62" width="0.1524" layer="91"/>
 <pinref part="R4" gate="G$1" pin="1"/>
-<wire x1="177.8" y1="2.54" x2="182.88" y2="2.54" width="0.1524" layer="91"/>
+<wire x1="177.8" y1="2.54" x2="195.58" y2="2.54" width="0.1524" layer="91"/>
 </segment>
 <segment>
@@
 <net name="RX" class="0">
 <segment>
-<pinref part="JP3" gate="JP" pin="P0/A0/TXD0"/>
-<wire x1="38.1" y1="55.88" x2="27.94" y2="55.88" width="0.1524" layer="91"/>
-<label x="27.94" y="55.88" size="1.27" layer="95" rot="R180" xref="yes"/>
-</segment>
-<segment>
 <pinref part="U$1" gate="G$1" pin="RX"/>
 <wire x1="165.1" y1="10.16" x2="172.72" y2="10.16" width="0.1524" layer="91"/>
 <label x="172.72" y="10.16" size="1.27" layer="95" xref="yes"/>
 </segment>
+<segment>
+<pinref part="JP3" gate="JP" pin="P2/A2/TXD1"/>
+<wire x1="38.1" y1="45.72" x2="27.94" y2="45.72" width="0.1524" layer="91"/>
+<label x="27.94" y="45.72" size="1.27" layer="95" ratio="15" rot="R180" xref="yes"/>
+</segment>
 </net>
 <net name="TX" class="0">
-<segment>
-<pinref part="JP3" gate="JP" pin="P1/A1/RXD0"/>
-<wire x1="38.1" y1="50.8" x2="27.94" y2="50.8" width="0.1524" layer="91"/>
-<label x="27.94" y="50.8" size="1.27" layer="95" rot="R180" xref="yes"/>
-</segment>
 <segment>
 <pinref part="U$1" gate="G$1" pin="TX"/>
@@
 <label x="172.72" y="12.7" size="1.27" layer="95" xref="yes"/>
 </segment>
+<segment>
+<pinref part="JP3" gate="JP" pin="P3/A3/RXD1"/>
+<wire x1="38.1" y1="40.64" x2="27.94" y2="40.64" width="0.1524" layer="91"/>
+<label x="27.94" y="40.64" size="1.27" layer="95" ratio="15" rot="R180" xref="yes"/>
+</segment>
 </net>
 <net name="P8" class="0">
@@
 <net name="RESET" class="0">
 <segment>
-<label x="198.12" y="10.16" size="1.27" layer="95" rot="R180" xref="yes"/>
+<label x="200.66" y="10.16" size="1.27" layer="95" rot="R180" xref="yes"/>
 <pinref part="S1" gate="G$1" pin="1"/>
-<wire x1="203.2" y1="10.16" x2="198.12" y2="10.16" width="0.1524" layer="91"/>
+<wire x1="203.2" y1="10.16" x2="200.66" y2="10.16" width="0.1524" layer="91"/>
 <pinref part="R2" gate="G$1" pin="1"/>
 <wire x1="203.2" y1="10.16" x2="203.2" y2="12.7" width="0.1524" layer="91"/>
@@
 <pinref part="R4" gate="G$1" pin="2"/>
 <wire x1="165.1" y1="2.54" x2="167.64" y2="2.54" width="0.1524" layer="91"/>
-<wire x1="167.64" y1="2.54" x2="167.64" y2="15.24" width="0.1524" layer="91"/>
+<wire x1="167.64" y1="2.54" x2="167.64" y2="25.4" width="0.1524" layer="91"/>
 <junction x="167.64" y="2.54"/>
-<pinref part="IO2" gate="G$1" pin="TP"/>
+<pinref part="U$2" gate="G$1" pin="1"/>
 </segment>
 </net>
@@
 <wire x1="132.08" y1="15.24" x2="132.08" y2="12.7" width="0.1524" layer="91"/>
 <junction x="132.08" y="12.7"/>
-<pinref part="RST" gate="G$1" pin="TP"/>
 <wire x1="132.08" y1="15.24" x2="106.68" y2="15.24" width="0.1524" layer="91"/>
-<junction x="132.08" y="15.24"/>
 <pinref part="JP1" gate="G$1" pin="1"/>
 <wire x1="106.68" y1="15.24" x2="106.68" y2="5.08" width="0.1524" layer="91"/>
 <wire x1="106.68" y1="5.08" x2="121.92" y2="5.08" width="0.1524" layer="91"/>
+<pinref part="U$3" gate="G$1" pin="1"/>
+<wire x1="132.08" y1="25.4" x2="132.08" y2="15.24" width="0.1524" layer="91"/>
+<junction x="132.08" y="15.24"/>
 </segment>
 </net>
@@
 </segment>
 </net>
+<net name="N$6" class="0">
+<segment>
+<pinref part="U$5" gate="G$1" pin="1"/>
+<pinref part="U$1" gate="G$1" pin="GPIO12"/>
+<wire x1="93.98" y1="0" x2="132.08" y2="0" width="0.1524" layer="91"/>
+</segment>
+</net>
+<net name="N$7" class="0">
+<segment>
+<pinref part="U$4" gate="G$1" pin="1"/>
+<pinref part="U$1" gate="G$1" pin="GPIO14"/>
+<wire x1="101.6" y1="2.54" x2="132.08" y2="2.54" width="0.1524" layer="91"/>
+</segment>
+</net>
+<net name="N$8" class="0">
+<segment>
+<pinref part="U$1" gate="G$1" pin="GPIO4"/>
+<pinref part="U$6" gate="G$1" pin="1"/>
+<wire x1="165.1" y1="7.62" x2="177.8" y2="7.62" width="0.1524" layer="91"/>
+<wire x1="177.8" y1="7.62" x2="177.8" y2="17.78" width="0.1524" layer="91"/>
+</segment>
+</net>
+<net name="N$9" class="0">
+<segment>
+<pinref part="U$1" gate="G$1" pin="GPIO5"/>
+<pinref part="U$7" gate="G$1" pin="1"/>
+<wire x1="165.1" y1="5.08" x2="185.42" y2="5.08" width="0.1524" layer="91"/>
+<wire x1="185.42" y1="5.08" x2="185.42" y2="22.86" width="0.1524" layer="91"/>
+</segment>
+</net>
+<net name="N$10" class="0">
+<segment>
+<pinref part="U$1" gate="G$1" pin="GPIO2"/>
+<pinref part="U$8" gate="G$1" pin="1"/>
+<wire x1="165.1" y1="0" x2="190.5" y2="0" width="0.1524" layer="91"/>
+<wire x1="190.5" y1="0" x2="190.5" y2="17.78" width="0.1524" layer="91"/>
+</segment>
+</net>

Commit message: Add files via upload
Parts:
- removed JP3: BC-MODULE-CORE, bigclown:BC-MODULE-CORE
- removed U$3, U$4, U$7: 1X1, headers_2mm:1X1
- added IO14, IO5, RST: 1X1, headers_2mm:1X1
- added JP2: BC-HEADER-MODULE-THT, bc-header:BC-HEADER-MODULE-THT
- R1: value 10k -> 1k
- renumbered U$2 to IO0, U$5 to IO12, U$6 to IO4, U$8 to IO2
Connections:
- net GND: now also JP2.GND; no longer JP3.GND
- net N$4: now also RST.1; no longer U$3.1
- net N$7: now also IO14.1; no longer U$4.1
- net N$9: now also IO5.1; no longer U$7.1
- net P6: now also JP2.P6/RTS1; no longer JP3.P6/RTS1
- net P7: now also JP2.P7/CTS1; no longer JP3.P7/CTS1
- net P8: now also JP2.P8; no longer JP3.P8
- net P9: now also JP2.P9; no longer JP3.P9
- net RX: now also JP2.P2/A2/TXD1; no longer JP3.P2/A2/TXD1
- net TX: now also JP2.P3/A3/RXD1; no longer JP3.P3/A3/RXD1
- net VCC: now also JP2.VDD; no longer JP3.VDD
Other:
- note added: "100u"
- note added: "220u"
- note added: "Made by chiptron.cz (2018)"
- note removed: "ESP02 - u.fl"
- note removed: "ESP03 - u.fl + pin"
- note removed: "ESP04 - pin"
- note removed: "chiptron.cz"
- moved on the sheet: CH_PD
